File: UA4C/vC3-WHITE FANG/Underdog.kicad_pcb (KiCad board)
At the start: 2 copper layers, 100 x 99.8 mm, 384 parts, among them IC2 IXDN602SIA, IC3 IXDN602SIA, J1 External MAP Conn, P1 INPUTS, P10 Dual VR C, P2 OUTPUTS, P3 SER0, P4 SER3, P5 SER2, P6 SPI0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

Commit message: Updated board layout files
Other:
- board text removed: "ASSEMBLED IN USA"
Changed lines of the file:
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@@
     (effects (font (size 0.5 1) (thickness 0.125)) (justify right mirror))
-  )
-  (gr_text "ASSEMBLED IN USA" (at 159.4 131.1) (layer F.SilkS)
-    (effects (font (size 1.25 1.25) (thickness 0.2)))
   )
   (gr_text "PRI-PRIMARY-RPM1-CRANK\nSEC-SECONDARY-RPM2-CAM\nDIGITAL 5V TRIGGER SET DIRECT\nANALOG (VR) OR HIGH VOLTAGE MUST USE TSC\nDIGITAL SIGNALS USUALLY REQUIRE PULL-UP\nSIGNAL CONDITIONERS INTEGRATE PULL-UP" (at 188 134.5) (layer B.SilkS)
